File: repositorio.kicad_sch (KiCad schematic)
At the start: 1 part, among them U1 ICM7555xB

Commit message: repositorio
Parts:
- removed U1: ICM7555xB, Package_SO:SOIC-8_3.9x4.9mm_P1.27mm, symbol Timer:ICM7555xB
- added M1: Module-knock-0.2, hellen-one-knock-0.2:knock, symbol knock:Module-knock-0.2
Changed lines of the file:
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@@
 	(paper "A4")
 	(symbol
-		(lib_id "Timer:ICM7555xB")
-		(at 111.76 59.69 0)
+		(lib_id "knock:Module-knock-0.2")
+		(at 83.82 59.69 0)
 		(unit 1)
 		(exclude_from_sim no)
@@
 		(dnp no)
 		(fields_autoplaced yes)
-		(property "Reference" "U1"
-			(at 113.9541 46.99 0)
+		(property "Reference" "M1"
+			(at 127 63.5314 0)
 			(effects
 				(font
 					(size 1.27 1.27)
 				)
-				(justify left)
 			)
 		)
-		(property "Value" "ICM7555xB"
-			(at 113.9541 49.53 0)
+		(property "Value" "Module-knock-0.2"
+			(at 127 66.0714 0)
 			(effects
 				(font
 					(size 1.27 1.27)
 				)
-				(justify left)
 			)
 		)
-		(property "Footprint" "Package_SO:SOIC-8_3.9x4.9mm_P1.27mm"
-			(at 133.35 69.85 0)
+		(property "Footprint" "hellen-one-knock-0.2:knock"
+			(at 83.82 59.69 0)
 			(effects
 				(font
@@
 			)
 		)
-		(property "Datasheet" "http://www.intersil.com/content/dam/Intersil/documents/icm7/icm7555-56.pdf"
-			(at 133.35 69.85 0)
+		(property "Datasheet" ""
+			(at 83.82 59.69 0)
 			(effects
 				(font
@@
 			)
 		)
-		(property "Description" "CMOS General Purpose Timer, 555 compatible, SOIC-8"
-			(at 111.76 59.69 0)
+		(property "Description" "Hellen-One Knock Pre-amplifier Module"
+			(at 83.82 59.69 0)
 			(effects
 				(font
@@
 			)
 		)
-		(pin "3"
+		(pin "E1"
 		)
-		(pin "4"
+		(pin "W2"
 		)
-		(pin "6"
+		(pin "E2"
 		)
-		(pin "7"
+		(pin "W1"
 		)
-		(pin "5"
-		)
-		(pin "8"
-		)
-		(pin "2"
-		)
-		(pin "1"
+		(pin "E3"
 		)
 		(instances
 			(project ""
 				(path "/57462394-f5e8-4e95-b2a6-e2c4782f3552"
-					(reference "U1")
+					(reference "M1")
 					(unit 1)
 				)
