File: repositorio.kicad_pcb (KiCad board)
At the start: 2 copper layers, 1 part, among them U1 ICM7555xB

Commit message: repositorio
Parts:
- added M1: Module-knock-0.2, hellen-one-knock-0.2:knock, F.Cu at (184.5, 80.2)

Commit message: repositorio
Parts:
- removed U1: ICM7555xB, Package_SO:SOIC-8_3.9x4.9mm_P1.27mm
Other:
- board outline added: 24 x 32 mm
